File: Ignignokt.kicad_sch (KiCad schematic)
At the start: 257 parts, among them J1 Barrel_Jack_Switch, J2 Conn_01x02_Pin, Q1 IRLB8721PBF, Q2 FQP27P06, U1 LM2585S-12, U2 LM2937ET-5.0, U3 PIC12F675-IMC

Commit message: Fix potentiometer issues
Screwed up the schematic for the potentiometers. The middle lead should be connected to power not the right lead. No lead should be connected to ground.

Signed-off-by: Nathan Hjelm <hjelmn@me.com>
Connections:
- net +12V: now also RV1.2; no longer RV1.1
- net +5V: now also RV2.2; no longer RV2.1
- net GND: no longer RV1.2, RV2.2
Changed lines of the file:
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@@
   (junction (at 54.61 144.78) (diameter 0) (color 0 0 0 0)
   )
-  (junction (at 135.89 171.45) (diameter 0) (color 0 0 0 0)
-  )
   (junction (at 80.01 144.78) (diameter 0) (color 0 0 0 0)
   )
@@
   (junction (at 13.97 93.98) (diameter 0) (color 0 0 0 0)
   )
+  (junction (at 139.7 167.64) (diameter 0) (color 0 0 0 0)
+  )
   (junction (at 68.58 161.29) (diameter 0) (color 0 0 0 0)
   )
@@
     (stroke (width 0) (type default))
   )
-  (wire (pts (xy 135.89 171.45) (xy 135.89 154.94))
-    (stroke (width 0) (type default))
-  )
   (wire (pts (xy 92.71 50.8) (xy 92.71 60.96))
     (stroke (width 0) (type default))
@@
     (stroke (width 0) (type default))
   )
+  (wire (pts (xy 172.72 154.94) (xy 139.7 154.94))
+    (stroke (width 0) (type default))
+  )
   (wire (pts (xy 118.11 116.84) (xy 133.35 116.84))
     (stroke (width 0) (type default))
@@
     (stroke (width 0) (type default))
   )
+  (wire (pts (xy 118.11 135.89) (xy 114.3 135.89))
+    (stroke (width 0) (type default))
+  )
   (wire (pts (xy 52.07 59.69) (xy 52.07 71.12))
     (stroke (width 0) (type default))
@@
     (stroke (width 0) (type default))
   )
-  (wire (pts (xy 127 171.45) (xy 135.89 171.45))
-    (stroke (width 0) (type default))
-  )
   (wire (pts (xy 198.12 173.99) (xy 199.39 173.99))
     (stroke (width 0) (type default))
@@
     (stroke (width 0) (type default))
   )
+  (wire (pts (xy 127 194.31) (xy 127 167.64))
+    (stroke (width 0) (type default))
+  )
   (wire (pts (xy 295.91 44.45) (xy 295.91 54.61))
     (stroke (width 0) (type default))
@@
     (stroke (width 0) (type default))
   )
+  (wire (pts (xy 127 167.64) (xy 139.7 167.64))
+    (stroke (width 0) (type default))
+  )
   (wire (pts (xy 95.25 49.53) (xy 95.25 60.96))
     (stroke (width 0) (type default))
@@
     (stroke (width 0) (type default))
   )
+  (wire (pts (xy 118.11 144.78) (xy 118.11 135.89))
+    (stroke (width 0) (type default))
+  )
   (wire (pts (xy 217.17 54.61) (xy 217.17 64.77))
     (stroke (width 0) (type default))
   )
-  (wire (pts (xy 135.89 154.94) (xy 172.72 154.94))
+  (wire (pts (xy 114.3 128.27) (xy 114.3 135.89))
     (stroke (width 0) (type default))
   )
@@
     (stroke (width 0) (type default))
   )
-  (wire (pts (xy 118.11 132.08) (xy 118.11 144.78))
-    (stroke (width 0) (type default))
-  )
   (wire (pts (xy 217.17 44.45) (xy 217.17 54.61))
     (stroke (width 0) (type default))
@@
     (stroke (width 0) (type default))
   )
+  (wire (pts (xy 139.7 154.94) (xy 139.7 167.64))
+    (stroke (width 0) (type default))
+  )
   (wire (pts (xy 40.64 120.65) (xy 45.72 120.65))
     (stroke (width 0) (type default))
@@
     (stroke (width 0) (type default))
   )
-  (wire (pts (xy 127 194.31) (xy 127 171.45))
-    (stroke (width 0) (type default))
-  )
   (wire (pts (xy 54.61 50.8) (xy 54.61 60.96))
     (stroke (width 0) (type default))
@@
     )
   )
-  (symbol (lib_id "power:GND") (at 114.3 128.27 270) (unit 1)
-    (in_bom yes) (on_board yes) (dnp no) (fields_autoplaced)
-    (property "Reference" "#PWR022" (at 107.95 128.27 0)
-      (effects (font (size 1.27 1.27)) hide)
-    )
-    (property "Value" "GND" (at 110.49 128.27 90)
-      (effects (font (size 1.27 1.27)) (justify right))
-    )
-    (property "Footprint" "" (at 114.3 128.27 0)
-      (effects (font (size 1.27 1.27)) hide)
-    )
-    (property "Datasheet" "" (at 114.3 128.27 0)
-      (effects (font (size 1.27 1.27)) hide)
-    )
-    (pin "1")
-    (instances
-      (project "Ignignokt"
-        (path "/f0a33db0-88ba-4d3e-9175-b5a39f1c39d8"
-          (reference "#PWR022") (unit 1)
-        )
-      )
-    )
-  )
   (symbol (lib_id "power:GND") (at 160.02 149.86 90) (unit 1)
     (in_bom yes) (on_board yes) (dnp no) (fields_autoplaced)
@@
         )
       )
-    )
-  )
-  (symbol (lib_id "power:GND") (at 139.7 167.64 180) (unit 1)
-    (in_bom yes) (on_board yes) (dnp no) (fields_autoplaced)
-    (property "Reference" "#PWR011" (at 139.7 161.29 0)
-      (effects (font (size 1.27 1.27)) hide)
-    )
-    (property "Value" "GND" (at 139.7 162.56 0)
-      (effects (font (size 1.27 1.27)))
-    )
-    (property "Footprint" "" (at 139.7 167.64 0)
-      (effects (font (size 1.27 1.27)) hide)
-    )
-    (property "Datasheet" "" (at 139.7 167.64 0)
-      (effects (font (size 1.27 1.27)) hide)
-    )
-    (pin "1")
-    (instances
-      (project "Ignignokt"
-        (path "/f0a33db0-88ba-4d3e-9175-b5a39f1c39d8"
-          (reference "#PWR011") (unit 1)
-        )
-      )

Commit message: Some minor tweaks
Moved the button light to between the light and ground instread of between power and the light. Cleaned up the schematic somewhat.

Signed-off-by: Nathan Hjelm <hjelmn@me.com>
Connections:
- net +5V: now also S1.E; no longer R50.2
- net GND: now also R50.1; no longer S1.F
- new net: R50.2, S1.F
Other:
- moved on the sheet: R50, RV1
Changed lines of the file:
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@@
   (junction (at 217.17 95.25) (diameter 0) (color 0 0 0 0)
   )
+  (junction (at 121.92 116.84) (diameter 0) (color 0 0 0 0)
+  )
   (junction (at 176.53 95.25) (diameter 0) (color 0 0 0 0)
   )
@@
   (junction (at 54.61 109.22) (diameter 0) (color 0 0 0 0)
   )
-  (junction (at 118.11 116.84) (diameter 0) (color 0 0 0 0)
-  )
   (junction (at 176.53 44.45) (diameter 0) (color 0 0 0 0)
   )
@@
   (junction (at 54.61 134.62) (diameter 0) (color 0 0 0 0)
   )
-  (wire (pts (xy 134.62 194.31) (xy 138.43 194.31))
+  (wire (pts (xy 127 194.31) (xy 138.43 194.31))
     (stroke (width 0) (type default))
   )
@@
     (stroke (width 0) (type default))
   )
-  (wire (pts (xy 118.11 116.84) (xy 118.11 124.46))
+  (wire (pts (xy 121.92 116.84) (xy 121.92 124.46))
     (stroke (width 0) (type default))
   )
@@
     (stroke (width 0) (type default))
   )
-  (wire (pts (xy 118.11 116.84) (xy 133.35 116.84))
-    (stroke (width 0) (type default))
-  )
   (wire (pts (xy 295.91 24.13) (xy 295.91 34.29))
     (stroke (width 0) (type default))
@@
     (stroke (width 0) (type default))
   )
-  (wire (pts (xy 118.11 135.89) (xy 114.3 135.89))
-    (stroke (width 0) (type default))
-  )
   (wire (pts (xy 52.07 59.69) (xy 52.07 71.12))
     (stroke (width 0) (type default))
@@
     (stroke (width 0) (type default))
   )
+  (wire (pts (xy 92.71 116.84) (xy 121.92 116.84))
+    (stroke (width 0) (type default))
+  )
+  (wire (pts (xy 121.92 116.84) (xy 133.35 116.84))
+    (stroke (width 0) (type default))
+  )
   (wire (pts (xy 217.17 95.25) (xy 217.17 105.41))
     (stroke (width 0) (type default))
@@
     (stroke (width 0) (type default))
   )
-  (wire (pts (xy 92.71 116.84) (xy 118.11 116.84))
-    (stroke (width 0) (type default))
-  )
   (wire (pts (xy 69.85 148.59) (xy 118.11 148.59))
     (stroke (width 0) (type default))
@@
     (stroke (width 0) (type default))
   )
-  (wire (pts (xy 118.11 144.78) (xy 118.11 135.89))
+  (wire (pts (xy 118.11 128.27) (xy 118.11 144.78))
     (stroke (width 0) (type default))
   )
   (wire (pts (xy 217.17 54.61) (xy 217.17 64.77))
-    (stroke (width 0) (type default))
-  )
-  (wire (pts (xy 114.3 128.27) (xy 114.3 135.89))
     (stroke (width 0) (type default))
   )
@@
     )
   )
-  (symbol (lib_id "Device:R_Potentiometer") (at 118.11 128.27 180) (unit 1)
-    (in_bom yes) (on_board yes) (dnp no) (fields_autoplaced)
-    (property "Reference" "RV1" (at 120.65 127 0)
+  (symbol (lib_id "Device:R_Potentiometer") (at 121.92 128.27 180) (unit 1)
+    (in_bom yes) (on_board yes) (dnp no) (fields_autoplaced)
+    (property "Reference" "RV1" (at 124.46 127 0)
       (effects (font (size 1.27 1.27)) (justify right))
     )
-    (property "Value" "1k" (at 120.65 129.54 0)
+    (property "Value" "1k" (at 124.46 129.54 0)
       (effects (font (size 1.27 1.27)) (justify right))
     )
-    (property "Footprint" "Potentiometer_THT:Potentiometer_Bourns_3299W_Vertical" (at 118.11 128.27 0)
-      (effects (font (size 1.27 1.27)) hide)
-    )
-    (property "Datasheet" "~" (at 118.11 128.27 0)
-      (effects (font (size 1.27 1.27)) hide)
-    )
-    (property "Part" "3299W-1-103LF" (at 118.11 128.27 0)
+    (property "Footprint" "Potentiometer_THT:Potentiometer_Bourns_3299W_Vertical" (at 121.92 128.27 0)
+      (effects (font (size 1.27 1.27)) hide)
+    )
+    (property "Datasheet" "~" (at 121.92 128.27 0)
+      (effects (font (size 1.27 1.27)) hide)
+    )
+    (property "Part" "3299W-1-103LF" (at 121.92 128.27 0)
       (effects (font (size 1.27 1.27)) hide)
     )
@@
     )
   )
-  (symbol (lib_id "power:GND") (at 153.67 194.31 90) (unit 1)
-    (in_bom yes) (on_board yes) (dnp no) (fields_autoplaced)
-    (property "Reference" "#PWR018" (at 160.02 194.31 0)
-      (effects (font (size 1.27 1.27)) hide)
-    )
-    (property "Value" "GND" (at 157.48 194.31 90)
+  (symbol (lib_id "power:GND") (at 161.29 194.31 90) (unit 1)
+    (in_bom yes) (on_board yes) (dnp no) (fields_autoplaced)
+    (property "Reference" "#PWR018" (at 167.64 194.31 0)
+      (effects (font (size 1.27 1.27)) hide)
+    )
+    (property "Value" "GND" (at 165.1 194.31 90)
       (effects (font (size 1.27 1.27)) (justify right))
     )
-    (property "Footprint" "" (at 153.67 194.31 0)
-      (effects (font (size 1.27 1.27)) hide)
-    )
-    (property "Datasheet" "" (at 153.67 194.31 0)
+    (property "Footprint" "" (at 161.29 194.31 0)
+      (effects (font (size 1.27 1.27)) hide)
+    )
+    (property "Datasheet" "" (at 161.29 194.31 0)
       (effects (font (size 1.27 1.27)) hide)
     )
@@
     )
   )
-  (symbol (lib_id "Device:R_US") (at 130.81 194.31 270) (unit 1)
-    (in_bom yes) (on_board yes) (dnp no) (fields_autoplaced)
-    (property "Reference" "R50" (at 130.81 187.96 90)
-      (effects (font (size 1.27 1.27)))
-    )
-    (property "Value" "200" (at 130.81 190.5 90)
-      (effects (font (size 1.27 1.27)))
-    )
-    (property "Footprint" "Resistor_THT:R_Axial_DIN0207_L6.3mm_D2.5mm_P10.16mm_Horizontal" (at 130.556 195.326 90)
-      (effects (font (size 1.27 1.27)) hide)
-    )
-    (property "Datasheet" "~" (at 130.81 194.31 0)
-      (effects (font (size 1.27 1.27)) hide)
-    )
+  (symbol (lib_id "Device:R_US") (at 157.48 194.31 270) (unit 1)
+    (in_bom yes) (on_board yes) (dnp no) (fields_autoplaced)
+    (property "Reference" "R50" (at 157.48 187.96 90)
+      (effects (font (size 1.27 1.27)))
+    )
+    (property "Value" "200" (at 157.48 190.5 90)
+      (effects (font (size 1.27 1.27)))
+    )
+    (property "Footprint" "Resistor_THT:R_Axial_DIN0207_L6.3mm_D2.5mm_P10.16mm_Horizontal" (at 157.226 195.326 90)
+      (effects (font (size 1.27 1.27)) hide)
+    )
+    (property "Datasheet" "~" (at 157.48 194.31 0)
+      (effects (font (size 1.27 1.27)) hide)
+    )
